Commit message: rb1_base_common/rb1_base_v3: Fix parent frame for top cover

File: rb1_base_common/rb1_base_description/urdf/bases/rb1_base_v3.urdf.xacro (robot description, xacro)
@@ -87,6 +87,6 @@
   </link>
   <joint name="${prefix}top_covert_joint" type="fixed">
-     <origin xyz="0.0 0.0 0.243" rpy="0 0 0 " />
-     <parent link="${prefix}base_footprint"/>
+     <origin xyz="0.0 0.0 0.0248" rpy="0 0 0 " />
+     <parent link="${prefix}base_link"/>
      <child link="${prefix}top_cover_link" />
   </joint>
